Commit message: added table urdf

File: Visual_Servoing/config/table.urdf (robot description, URDF)
Before this commit: robot rectangular_block, 1 links, 1 joints
Links:
- removed link base_link
- added link cube, mass 1.0; collision box size=1 1 1; visual box size=0.1 0.1 0.1
Joints:
- removed joint fixed
