Commit message: added blender objects

File: Multi_Agent_RL_Dexterous_Manipulation/config/assets/triangle.urdf (robot description, URDF)
Before this commit: robot triangle_block, 1 links, 0 joints
Links:
- link block: geometry collision mesh filename=./config/assets/triangle.dae; visual mesh filename=./config/assets/triangle.dae
