Commit message: fixed vs bug and disc is ready for training!

File: Multi_Agent_RL_Dexterous_Manipulation/config/assets/disc.urdf (robot description, URDF)
Before this commit: robot disc, 1 links, 0 joints
Links:
- link disc: mass 1.0 -> None; geometry collision cylinder length=0.001 radius=0.035; collision cylinder length=0.019 radius=0.035
Joints:
- added joint bottom_disk_to_side_joint: type fixed, parent side_link, child bottom_disk_link, origin xyz=0 0 -0.0095 rpy=0 0 0

Commit message: started adding blender files

File: Multi_Agent_RL_Dexterous_Manipulation/config/assets/disc.urdf (robot description, URDF)
Before this commit: robot disc, 1 links, 1 joints
Joints:
- removed joint bottom_disk_to_side_joint

Commit message: Commit before big change in codebase to include multiple objects

File: Multi_Agent_RL_Dexterous_Manipulation/config/assets/disc.urdf (robot description, URDF)
Before this commit: robot disc, 1 links, 0 joints
Joints:
- added joint bottom_disk_to_side_joint: type fixed, parent side_link, child bottom_disk_link, origin xyz=0 0 -0.0095 rpy=0 0 0
