Commit message: Major Overhaul added 9 objects and faster bd_pts code

File: Multi_Agent_RL_Dexterous_Manipulation/config/table.urdf (robot description, URDF)
Before this commit: robot table, 1 links, 0 joints
Links:
- link cube: geometry collision box size=2 2 1; visual box size=0.1 0.1 0.1

Commit message: fixed transformation bugs

File: Multi_Agent_RL_Dexterous_Manipulation/config/table.urdf (robot description, URDF)
Before this commit: robot table, 1 links, 0 joints
Links:
- link cube: geometry collision box size=1 1 1; visual box size=0.1 0.1 0.1
